Commit message: 使用圆柱描述轮子碰撞属性，缩小hip关节的惩罚阈值，纠正hip关节位置

File: resources/robots/tita/urdf/tita_v618.urdf (robot description, URDF)
Before this commit: robot tita_v618, 9 links, 8 joints
Links:
- link left_wheel: geometry collision cylinder length=0.034 radius=0.0925; visual mesh filename=../meshes/left_wheel.STL
- link right_wheel: geometry collision cylinder length=0.034 radius=0.0925; visual mesh filename=../meshes/right_wheel.STL
Joints:
- joint joint_left_wheel: limit effort=10 velocity=104.88 -> lower=-6.283185e4 upper=6.283185e4 effort=10 velocity=104.88
- joint joint_right_wheel: limit effort=10 velocity=104.88 -> lower=-6.283185e4 upper=6.283185e4 effort=10 velocity=104.88

Commit message: 注意：轮子位置限制在绝对值-2pai到2pai中，第一版可行的上楼梯版本

File: resources/robots/tita/urdf/tita_v618.urdf (robot description, URDF)
Before this commit: robot tita_v618, 9 links, 8 joints
Joints:
- joint joint_left_wheel: limit lower=-6.283185e4 upper=6.283185e4 effort=10 velocity=104.88 -> effort=10 velocity=104.88
- joint joint_right_wheel: limit lower=-6.283185e4 upper=6.283185e4 effort=10 velocity=104.88 -> effort=10 velocity=104.88
